File: work_table_light/work_table_light.sch (EAGLE design)
At the start: 8 parts, among them IC1 TINY24/44/84-PU

Commit message: Basic Schematic Finished
Connections:
- removed net N$1: IC1.(PCINT6/OC1A/SDA/MOSI/ADC6)PA6, JP1.1
- removed net N$4: IC1.(PCINT4/T1/SCL/USCK/ADC4)PA4, JP1.3
- new net PA4: JP1.3
- new net PA5: JP1.1
- new net PA6: JP1.4
- new net PB3: JP1.5
- net N$5: no longer JP1.5
Changed lines of the file:
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@@
-</segment>
-</net>
-<net name="N$4" class="0">
-<segment>
-<pinref part="JP1" gate="G$1" pin="3"/>
-<wire x1="66.04" y1="22.86" x2="88.9" y2="22.86" width="0.1524" layer="91"/>
-<pinref part="IC1" gate="1" pin="(PCINT4/T1/SCL/USCK/ADC4)PA4"/>
-<wire x1="88.9" y1="22.86" x2="88.9" y2="50.8" width="0.1524" layer="91"/>
-<wire x1="88.9" y1="50.8" x2="86.36" y2="50.8" width="0.1524" layer="91"/>
 </segment>
 </net>
@@
 <pinref part="IC1" gate="1" pin="(PCINT11/RESET/DW)PB3"/>
 <wire x1="86.36" y1="73.66" x2="86.36" y2="71.12" width="0.1524" layer="91"/>
-<wire x1="116.84" y1="71.12" x2="86.36" y2="71.12" width="0.1524" layer="91"/>
-<junction x="86.36" y="71.12"/>
-<pinref part="JP1" gate="G$1" pin="5"/>
-<wire x1="66.04" y1="25.4" x2="116.84" y2="25.4" width="0.1524" layer="91"/>
-<wire x1="116.84" y1="25.4" x2="116.84" y2="71.12" width="0.1524" layer="91"/>
-</segment>
-</net>
-<net name="N$1" class="0">
-<segment>
-<pinref part="JP1" gate="G$1" pin="1"/>
-<pinref part="IC1" gate="1" pin="(PCINT6/OC1A/SDA/MOSI/ADC6)PA6"/>
-<wire x1="66.04" y1="20.32" x2="86.36" y2="20.32" width="0.1524" layer="91"/>
-<wire x1="86.36" y1="20.32" x2="86.36" y2="55.88" width="0.1524" layer="91"/>
 </segment>
 </net>
@@
 </segment>
 </net>
+<net name="PB3" class="0">
+<segment>
+<pinref part="JP1" gate="G$1" pin="5"/>
+<wire x1="66.04" y1="25.4" x2="83.82" y2="25.4" width="0.1524" layer="91"/>
+<label x="83.82" y="25.4" size="1.778" layer="95"/>
+</segment>
+</net>
+<net name="PA4" class="0">
+<segment>
+<pinref part="JP1" gate="G$1" pin="3"/>
+<wire x1="66.04" y1="22.86" x2="83.82" y2="22.86" width="0.1524" layer="91"/>
+<label x="83.82" y="22.86" size="1.778" layer="95"/>
+</segment>
+</net>
+<net name="PA5" class="0">
+<segment>
+<pinref part="JP1" gate="G$1" pin="1"/>
+<wire x1="66.04" y1="20.32" x2="83.82" y2="20.32" width="0.1524" layer="91"/>
+<label x="83.82" y="20.32" size="1.778" layer="95"/>
+</segment>
+</net>
+<net name="PA6" class="0">
+<segment>
+<pinref part="JP1" gate="G$1" pin="4"/>
+<wire x1="55.88" y1="22.86" x2="40.64" y2="22.86" width="0.1524" layer="91"/>
+<label x="40.64" y="22.86" size="1.778" layer="95"/>
+</segment>
+</net>

Commit message: schematic updated
Parts:
- removed JP1: AVR-ISP-6VERT, avr-7:AVR-ISP-6VERT
- added DZ1, DZ2, DZ3: LZR183, led:LZR183
- added LED3: F50360, led:F50360
- added Q1, Q2, Q3: IRFP250, transistor-power:IRFP250
- added R3: (no value), rcl:POTENTIOMETER_PT-10S
- added T1, T2, T3: 2N3904, transistor:2N3904
- LED1, LED2: value (none) -> F50360; device eagle-ltspice:LED_ELD260 -> led:F50360
Connections:
- removed net PA1: R2.3
- removed net PA4: JP1.3
- removed net PA5: JP1.1
- removed net PA6: JP1.4
- removed net PB3: JP1.5
- new net N$1: LED1.RC, LED2.RC, LED3.RC, T1.C
- new net N$10: Q3.S
- new net N$11: DZ1-1.A, Q1.D
- new net N$12: DZ1-1.C, DZ2-1.A
- new net N$13: DZ2-1.C, DZ3-1.A
- new net N$14: DZ1-2.A, Q2.D
- new net N$15: DZ1-2.C, DZ2-2.A
- new net N$16: DZ2-2.C, DZ3-2.A
- new net N$17: DZ1-3.A, Q3.D
- new net N$18: DZ1-3.C, DZ2-3.A
- new net N$19: DZ2-3.C, DZ3-3.A
- new net N$20: IC1.(PCINT10/INT0/OC0A/CKOUT)PB2, T1.B
- new net N$21: LED1.GC, LED2.GC, LED3.GC, T2.C
- new net N$22: LED1.BC, LED2.BC, LED3.BC, T3.C
- new net N$23: IC1.(PCINT1/AIN0/ADC1)PA1, R2.3
- new net N$4: IC1.(PCINT6/OC1A/SDA/MOSI/ADC6)PA6, T3.B
- new net N$5: IC1.(PCINT7/ICP/OC0B/ADC7)PA7, T2.B
- new net N$6: IC1.(PCINT2/AIN1/ADC2)PA2, R3.3
- new net N$7: Q1.S
- new net N$8: Q2.S
- net GND: now also R3.2, T1.E, T2.E, T3.E; no longer JP1.6, LED1.C, LED2.C
- net N$2: now also Q1.G, Q2.G, Q3.G; no longer LED1.A, LED2.A
- net VCC: now also DZ3-1.C, DZ3-2.C, DZ3-3.C, LED1.BA, LED1.GA, LED1.RA, LED2.BA, LED2.GA, LED2.RA, LED3.BA, LED3.GA, LED3.RA, R3.1; no longer JP1.2
Other:
- moved on the sheet: C2, R2

Commit message: schematic updated
Parts:
- added JP1: AVR-ISP-6VERT, avr-7:AVR-ISP-6VERT
Connections:
- new net PA4: JP1.3
- new net PA5: JP1.1
- new net PA6: JP1.4
- new net PB3: JP1.5
- net GND: now also JP1.6
- net VCC: now also JP1.2
Other:
- moved on the sheet: DZ1-1, DZ1-2, DZ1-3, DZ2-1, DZ2-2, DZ2-3, DZ3-1, DZ3-2, DZ3-3, LED1, LED2, LED3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

Commit message: updated schematic
Parts:
- added S5, S6: (no value), eswitch-tact:TL3302-J
Connections:
- net N$1 renamed RED
- net N$2 renamed PA5(OC1B,MISO)
- net N$20 renamed PB2(OC0A)
- net N$21 renamed GREEN
- net N$23 renamed PA1(PCINT1)
- net N$4 renamed PA6(OC1A,MOSI)
- net N$5 renamed PA7(OCOB)
- net N$6 renamed PA2(PCINT2)
- net N$9 renamed RESET
- removed net N$22: LED1.BC, LED2.BC, LED3.BC, T3.C
- new net BLUE: LED3.BC, T3.C
- new net N$1: T1.E, T2.E, T3.E
- new net N$21: LED1.BC, LED2.BC
- new net PA4(SCK): IC1.(PCINT4/T1/SCL/USCK/ADC4)PA4
- new net PB0(SWITCH1): IC1.(PCINT9/XTAL2)PB1, S5.1
- new net PB1(SWITCH2): IC1.(PCINT8/XTAL1/CLKI)PB0, S6.1
- net GND: now also S5.2, S6.2; no longer T1.E, T2.E, T3.E
- net N$11: now also Q3.D; no longer Q1.D
- net N$17: now also Q1.D; no longer Q3.D
Other:
- note added: "Potentiometers used to dim the white led strips and scroll through the colors of the RGB led strip"
- note added: "Push buttons for the different modes of the work table light"
- note added: "This section is the RGB portion of the work table light. The transistors are 2N3904, however the RGB leds in the schematic are not the same model used in practice. In practice a 5050 RGB led strip is used"
- note added: "This section of the schematic is the main white light for work table light. The MOSFETs used in practice are FQP30N06L. The leds used in practice are 3014 white led strips with 204 leds/m."
- moved on the sheet: DZ1-1, DZ1-2, DZ1-3, DZ2-1, DZ2-2, DZ2-3, DZ3-1, DZ3-2, DZ3-3, JP1, LED1, LED2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

Commit message: updated schematic
Parts:
- added U$1: FRAME_AUTH, frame_with_author:FRAME_AUTH
Changed lines of the file:
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@@
 <part name="S6" library="eswitch-tact" deviceset="TL3302" device="-J"/>
 <part name="GND8" library="supply1" library_urn="urn:adsk.eagle:library:371" deviceset="GND" device=""/>
+<part name="U$1" library="frame_with_author" deviceset="FRAME_AUTH" device=""/>
 </parts>
 <sheets>
@@
 <instance part="S6" gate="G$1" x="127" y="81.28"/>
 <instance part="GND8" gate="1" x="132.08" y="76.2"/>
+<instance part="U$1" gate="G$1" x="-55.88" y="-76.2"/>
 </instances>
 <busses>

Commit message: updated schematic
Parts:
- removed C1, C2: (no value), capacitor-wima:C2,5-3
- removed T1, T2, T3: 2N3904, transistor:2N3904
- added C3, C4: 1uF, adafruit:C-US025-024X044
- added C5, C6: 10uF, adafruit:C-US025-024X044
- added Q4, Q6, Q7: IRFP250, transistor-power:IRFP250
- added R10, R11, R12, R13, R14, R15: (no value), rcl:R-US_0204/5
- added R16, R18: 10K, pot:TRIM_US-CIP20C-6MM
- added R4, R5, R6, R7, R8, R9: 220K, resistor:R-US_0207/10
- R2, R3: value (none) -> 220K; device rcl:POTENTIOMETER_PT-10S -> resistor:R-US_0207/10; SPICEMODEL 1K -> (none)
Connections:
- removed net BLUE: LED3.BC, T3.C
- removed net GREEN: LED1.GC, LED2.GC, LED3.GC, T2.C
- removed net RED: LED1.RC, LED2.RC, LED3.RC, T1.C
- new net BLUE(OC1A,PA6): LED3.BC, Q6.D, R7.2
- new net GREEN(OC0B,PA7): LED1.GC, LED2.GC, LED3.GC, Q7.D, R8.2
- new net N$2: Q1.S, R5.1
- new net N$20: Q3.G, R15.2
- new net N$22: R18.S, R3.1
- new net N$23: R16.S, R2.1
- new net N$4: Q2.S, R4.1
- new net N$5: Q3.S, R6.1
- new net N$6: Q7.G, R11.2
- new net N$9: Q2.G, R14.2
- new net RED(PB2,OCOA): LED1.RC, LED2.RC, LED3.RC, Q4.D, R9.2
- net GND: now also C3.2, C4.2, C5.2, C6.2, R16.E, R18.E; no longer C1.2, C2.2, R2.2, R3.2
- net N$1: now also Q4.G, R10.2; no longer T1.E, T2.E, T3.E
- net N$10: now also Q4.S, Q6.S, Q7.S, R7.1, R8.1, R9.1; no longer Q3.S
- net N$11: now also R6.2
- net N$14: now also R4.2
- net N$17: now also R5.2
- net N$3: now also C6.1; no longer C2.1
- net N$7: now also Q1.G, R13.2; no longer Q1.S
- net N$8: now also Q6.G, R12.2; no longer Q2.S
- net PA1(PCINT1): now also C3.1, R2.2; no longer R2.3
- net PA2(PCINT2): now also C4.1, R3.2; no longer R3.3
- net PA5(OC1B,MISO): now also R13.1, R14.1, R15.1; no longer Q1.G, Q2.G, Q3.G
- net PA6(OC1A,MOSI): now also R12.1; no longer T3.B
- net PA7(OCOB): now also R11.1; no longer T2.B
- net PB2(OC0A): now also R10.1; no longer T1.B
- net VCC: now also C5.1, R16.A, R18.A; no longer C1.1, R2.1, R3.1
Other:
- note added: "Potentiometers used to dim the white led strips and scroll through the colors of the RGB led strip The values of R2 and R3 are still being experimented with."
- note added: "This section is the RGB portion of the work table light. The mosfets being used are the same as ones used for the white light (FQP30N06L), however the RGB leds in the schematic are not the same model used in practice. In practice a 5050 RGB led strip is used"
- note removed: "Potentiometers used to dim the white led strips and scroll through the colors of the RGB led strip"
- note removed: "This section is the RGB portion of the work table light. The transistors are 2N3904, however the RGB leds in the schematic are not the same model used in practice. In practice a 5050 RGB led strip is used"
- moved on the sheet: DZ1-1, DZ1-2, DZ1-3, DZ2-1, DZ2-2, DZ2-3, DZ3-1, DZ3-2, DZ3-3, LED1, LED2, LED3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

Commit message: updated schematic
Parts:
- removed Q2, Q3: IRFP250, transistor-power:IRFP250
- removed R14, R15: (no value), rcl:R-US_0204/5
- removed R4, R6: 220K, resistor:R-US_0207/10
Connections:
- removed net N$14: DZ1-2.A, Q2.D, R4.2
- removed net N$17: DZ1-3.A, Q1.D, R5.2
- removed net N$20: Q3.G, R15.2
- removed net N$9: Q2.G, R14.2
- net GND: now also Q1.S, R5.1
- net N$11: now also Q1.D, R5.2; no longer DZ1-1.A, Q3.D, R6.2
- net N$2: now also DZ1-3.A; no longer Q1.S, R5.1
- net N$4: now also DZ1-2.A; no longer Q2.S, R4.1
- net N$5: now also DZ1-1.A; no longer Q3.S, R6.1
- net PA5(OC1B,MISO): no longer R14.1, R15.1
Other:
- moved on the sheet: S1, S2, S3

Commit message: updated schematic
Connections:
- removed net N$12: DZ1-1.C, DZ2-1.A
- removed net N$13: DZ2-1.C, DZ3-1.A
- removed net N$15: DZ1-2.C, DZ2-2.A
- removed net N$16: DZ2-2.C, DZ3-2.A
- removed net N$18: DZ1-3.C, DZ2-3.A
- removed net N$19: DZ2-3.C, DZ3-3.A
- net N$2: now also DZ2-3.A, DZ3-3.A
- net N$4: now also DZ2-2.A, DZ3-2.A
- net N$5: now also DZ2-1.A, DZ3-1.A
- net VCC: now also DZ1-1.C, DZ1-2.C, DZ1-3.C, DZ2-1.C, DZ2-2.C, DZ2-3.C
Changed lines of the file:
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@@
 <wire x1="289.56" y1="17.78" x2="297.18" y2="17.78" width="0.1524" layer="91"/>
 <wire x1="297.18" y1="17.78" x2="297.18" y2="38.1" width="0.1524" layer="91"/>
+<pinref part="DZ2" gate="-3" pin="C"/>
+<wire x1="269.24" y1="30.48" x2="269.24" y2="33.02" width="0.1524" layer="91"/>
+<wire x1="269.24" y1="33.02" x2="287.02" y2="33.02" width="0.1524" layer="91"/>
+<wire x1="287.02" y1="33.02" x2="287.02" y2="30.48" width="0.1524" layer="91"/>
+<junction x="287.02" y="30.48"/>
+<pinref part="DZ1" gate="-3" pin="C"/>
+<wire x1="251.46" y1="30.48" x2="251.46" y2="33.02" width="0.1524" layer="91"/>
+<wire x1="251.46" y1="33.02" x2="269.24" y2="33.02" width="0.1524" layer="91"/>
+<junction x="269.24" y="33.02"/>
+<pinref part="DZ2" gate="-2" pin="C"/>
+<wire x1="269.24" y1="17.78" x2="269.24" y2="20.32" width="0.1524" layer="91"/>
+<wire x1="269.24" y1="20.32" x2="287.02" y2="20.32" width="0.1524" layer="91"/>
+<wire x1="287.02" y1="20.32" x2="287.02" y2="17.78" width="0.1524" layer="91"/>
+<junction x="287.02" y="17.78"/>
+<pinref part="DZ1" gate="-2" pin="C"/>
+<wire x1="251.46" y1="17.78" x2="251.46" y2="20.32" width="0.1524" layer="91"/>
+<wire x1="251.46" y1="20.32" x2="269.24" y2="20.32" width="0.1524" layer="91"/>
+<junction x="269.24" y="20.32"/>
+<pinref part="DZ2" gate="-1" pin="C"/>
+<wire x1="269.24" y1="5.08" x2="269.24" y2="7.62" width="0.1524" layer="91"/>
+<wire x1="269.24" y1="7.62" x2="287.02" y2="7.62" width="0.1524" layer="91"/>
+<wire x1="287.02" y1="7.62" x2="287.02" y2="5.08" width="0.1524" layer="91"/>
+<junction x="287.02" y="5.08"/>
+<pinref part="DZ1" gate="-1" pin="C"/>
+<wire x1="251.46" y1="5.08" x2="251.46" y2="7.62" width="0.1524" layer="91"/>
+<wire x1="251.46" y1="7.62" x2="269.24" y2="7.62" width="0.1524" layer="91"/>
+<junction x="269.24" y="7.62"/>
 </segment>
 </net>
@@
 <label x="86.36" y="53.34" size="1.778" layer="95"/>
 <wire x1="154.94" y1="53.34" x2="154.94" y2="30.48" width="0.1524" layer="91"/>
-</segment>
-</net>
-<net name="N$12" class="0">
-<segment>
-<pinref part="DZ1" gate="-1" pin="C"/>
-<pinref part="DZ2" gate="-1" pin="A"/>
-<wire x1="251.46" y1="5.08" x2="261.62" y2="5.08" width="0.1524" layer="91"/>
-</segment>
-</net>
-<net name="N$13" class="0">
-<segment>
-<pinref part="DZ2" gate="-1" pin="C"/>
-<pinref part="DZ3" gate="-1" pin="A"/>
-<wire x1="269.24" y1="5.08" x2="279.4" y2="5.08" width="0.1524" layer="91"/>
-</segment>
-</net>
-<net name="N$15" class="0">
-<segment>
-<pinref part="DZ1" gate="-2" pin="C"/>
-<pinref part="DZ2" gate="-2" pin="A"/>
-<wire x1="251.46" y1="17.78" x2="261.62" y2="17.78" width="0.1524" layer="91"/>
-</segment>
-</net>
-<net name="N$16" class="0">
-<segment>
-<pinref part="DZ2" gate="-2" pin="C"/>
-<pinref part="DZ3" gate="-2" pin="A"/>
-<wire x1="269.24" y1="17.78" x2="279.4" y2="17.78" width="0.1524" layer="91"/>
-</segment>
-</net>
-<net name="N$18" class="0">
-<segment>
-<pinref part="DZ1" gate="-3" pin="C"/>
-<pinref part="DZ2" gate="-3" pin="A"/>
-<wire x1="251.46" y1="30.48" x2="261.62" y2="30.48" width="0.1524" layer="91"/>
-</segment>
-</net>
-<net name="N$19" class="0">
-<segment>
-<pinref part="DZ2" gate="-3" pin="C"/>
-<pinref part="DZ3" gate="-3" pin="A"/>
-<wire x1="269.24" y1="30.48" x2="279.4" y2="30.48" width="0.1524" layer="91"/>
 </segment>
 </net>
@@
 <pinref part="DZ1" gate="-3" pin="A"/>
 <wire x1="243.84" y1="30.48" x2="236.22" y2="30.48" width="0.1524" layer="91"/>
+<pinref part="DZ2" gate="-3" pin="A"/>
+<wire x1="261.62" y1="30.48" x2="261.62" y2="27.94" width="0.1524" layer="91"/>
+<wire x1="261.62" y1="27.94" x2="243.84" y2="27.94" width="0.1524" layer="91"/>
+<wire x1="243.84" y1="27.94" x2="243.84" y2="30.48" width="0.1524" layer="91"/>
+<junction x="243.84" y="30.48"/>
+<pinref part="DZ3" gate="-3" pin="A"/>
+<wire x1="279.4" y1="30.48" x2="279.4" y2="27.94" width="0.1524" layer="91"/>
+<wire x1="279.4" y1="27.94" x2="261.62" y2="27.94" width="0.1524" layer="91"/>
+<junction x="261.62" y="27.94"/>
 </segment>
 </net>
@@
 <pinref part="DZ1" gate="-2" pin="A"/>
 <wire x1="243.84" y1="17.78" x2="236.22" y2="17.78" width="0.1524" layer="91"/>
+<pinref part="DZ2" gate="-2" pin="A"/>
+<wire x1="261.62" y1="17.78" x2="261.62" y2="15.24" width="0.1524" layer="91"/>
+<wire x1="261.62" y1="15.24" x2="243.84" y2="15.24" width="0.1524" layer="91"/>
+<wire x1="243.84" y1="15.24" x2="243.84" y2="17.78" width="0.1524" layer="91"/>
+<junction x="243.84" y="17.78"/>
+<pinref part="DZ3" gate="-2" pin="A"/>
+<wire x1="279.4" y1="17.78" x2="279.4" y2="15.24" width="0.1524" layer="91"/>
+<wire x1="279.4" y1="15.24" x2="261.62" y2="15.24" width="0.1524" layer="91"/>
+<junction x="261.62" y="15.24"/>
 </segment>
 </net>
@@
 <pinref part="DZ1" gate="-1" pin="A"/>
 <wire x1="243.84" y1="5.08" x2="236.22" y2="5.08" width="0.1524" layer="91"/>
-</segment>
-</net>
+<pinref part="DZ2" gate="-1" pin="A"/>
+<wire x1="261.62" y1="5.08" x2="261.62" y2="2.54" width="0.1524" layer="91"/>
+<wire x1="261.62" y1="2.54" x2="243.84" y2="2.54" width="0.1524" layer="91"/>
+<wire x1="243.84" y1="2.54" x2="243.84" y2="5.08" width="0.1524" layer="91"/>
+<junction x="243.84" y="5.08"/>
+<pinref part="DZ3" gate="-1" pin="A"/>
+<wire x1="279.4" y1="5.08" x2="279.4" y2="2.54" width="0.1524" layer="91"/>
+<wire x1="279.4" y1="2.54" x2="261.62" y2="2.54" width="0.1524" layer="91"/>
+<junction x="261.62" y="2.54"/>
+</segment>
+</net>
